File: KiCAD/music_box.sch (KiCad schematic (older format))
At the start: 12 parts, among them Q1 2N3904, SW1 power, SW2 play, U1 PIC10F202-I_P

Commit message: premier commit
Parts:
- removed C3: 470µF, symbol device:CP
- added D1: LED, symbol device:LED
- added LS1: 135R, symbol device:Speaker
- added R1: 470R, symbol device:R
- added R2: 33k, symbol device:R
- BT1: value CR2250 -> 4,5Volt
- C2: value 22µF -> 33µF
- LS2: renamed from LS1; value Speaker_Crystal -> piezo
- renumbered R1 to R3, R2 to R4, R3 to R5
Connections:
- net GND: now also LS1.2
- net +Vdd: now reaches C1.2, SW1.2 (B), U1.2 (VDD)
- net +Vdd: now also R1.2, R2.2
- net at U1.3 (T0CKI/FOSC4/GP2): now also D1.1 (K); no longer SW2.2
- net at U1.8 (Vpp/~MCLR~/GP3): now also SW2.2, R2.1
- net Eq1: now reaches Q1.3 (E), R5.2
- net Eq1: now also LS2.1, LS1.1
- new net: D1.2 (A), R1.1
Other:
- note added: "boite à musique"
- note added: "durée de l'attaque 5*R1*C2\ndurée du déclin 5*(R2+GRe)*C2"
- note added: "option 2\n"
- moved on the sheet: LS2, R5, SW2
Changed lines of the file:
@@
 P 3500 3525
 F 0 "BT1" H 3608 3571 50  0000 L CNN
-F 1 "CR2250" H 3608 3480 50  0000 L CNN
+F 1 "4,5Volt" H 3608 3480 50  0000 L CNN
 F 2 "" V 3500 3585 50  0001 C CNN
 F 3 "~" V 3500 3585 50  0001 C CNN
@@
 $EndComp
 $Comp
-L device:R R2
+L device:R R4
 U 1 1 5BFF3B9C
 P 6150 3425
-F 0 "R2" V 5943 3425 50  0000 C CNN
+F 0 "R4" V 5943 3425 50  0000 C CNN
 F 1 "3K" V 6034 3425 50  0000 C CNN
 F 2 "" V 6080 3425 50  0001 C CNN
@@
 $EndComp
 $Comp
-L device:R R1
+L device:R R3
 U 1 1 5BFF3BDE
 P 5750 3425
-F 0 "R1" V 5543 3425 50  0000 C CNN
+F 0 "R3" V 5543 3425 50  0000 C CNN
 F 1 "470R" V 5634 3425 50  0000 C CNN
 F 2 "" V 5680 3425 50  0001 C CNN
@@
 $EndComp
 $Comp
-L device:R R3
+L device:R R5
 U 1 1 5BFF3C9C
-P 6750 3850
-F 0 "R3" H 6680 3804 50  0000 R CNN
-F 1 "120R" H 6680 3895 50  0000 R CNN
-F 2 "" V 6680 3850 50  0001 C CNN
-F 3 "" H 6750 3850 50  0001 C CNN
-	1    6750 3850
+P 7775 4000
+F 0 "R5" H 7705 3954 50  0000 R CNN
+F 1 "120R" H 7705 4045 50  0000 R CNN
+F 2 "" V 7705 4000 50  0001 C CNN
+F 3 "" H 7775 4000 50  0001 C CNN
+	1    7775 4000
 	-1   0    0    1
 $EndComp
@@
 $EndComp
 $Comp
-L power:GND #PWR04
+L power:GND #PWR05
 U 1 1 5BFF4120
-P 6750 4000
-F 0 "#PWR04" H 6750 3750 50  0001 C CNN
-F 1 "GND" H 6755 3827 50  0000 C CNN
-F 2 "" H 6750 4000 50  0001 C CNN
-F 3 "" H 6750 4000 50  0001 C CNN
-	1    6750 4000
-	1    0    0    -1
-$EndComp
-Wire Wire Line
-	6750 3625 6750 3650
-$Comp
-L device:CP C3
-U 1 1 5BFF4221
-P 7150 3650
-F 0 "C3" V 7405 3650 50  0000 C CNN
-F 1 "470µF" V 7314 3650 50  0000 C CNN
-F 2 "" H 7188 3500 50  0001 C CNN
-F 3 "" H 7150 3650 50  0001 C CNN
-	1    7150 3650
-	0    -1   -1   0
-$EndComp
-$Comp
-L device:Speaker_Crystal LS1
+P 7775 4150
+F 0 "#PWR05" H 7775 3900 50  0001 C CNN
+F 1 "GND" H 7780 3977 50  0000 C CNN
+F 2 "" H 7775 4150 50  0001 C CNN
+F 3 "" H 7775 4150 50  0001 C CNN
+	1    7775 4150
+	1    0    0    -1
+$EndComp
+Wire Wire Line
+	7775 3775 7775 3800
+$Comp
+L device:Speaker_Crystal LS2
 U 1 1 5BFF43B0
-P 7550 3650
-F 0 "LS1" H 7725 3646 50  0000 L CNN
-F 1 "Speaker_Crystal" H 7725 3555 50  0000 L CNN
-F 2 "" H 7515 3600 50  0001 C CNN
-F 3 "" H 7515 3600 50  0001 C CNN
-	1    7550 3650
-	1    0    0    -1
-$EndComp
-Wire Wire Line
-	7300 3650 7350 3650
-Wire Wire Line
-	7000 3650 6750 3650
-Connection ~ 6750 3650
-Wire Wire Line
-	6750 3650 6750 3700
+P 8575 3800
+F 0 "LS2" H 8750 3796 50  0000 L CNN
+F 1 "piezo" H 8750 3705 50  0000 L CNN
+F 2 "" H 8540 3750 50  0001 C CNN
+F 3 "" H 8540 3750 50  0001 C CNN
+	1    8575 3800
+	1    0    0    -1
+$EndComp
+Connection ~ 7775 3800
+Wire Wire Line
+	7775 3800 7775 3850
 Wire Wire Line
 	6750 3225 6750 3125
@@
 L switches:SW_Push SW2
 U 1 1 5BFF479A
-P 5650 4225
-F 0 "SW2" V 5696 4177 50  0000 R CNN
-F 1 "play" V 5605 4177 50  0000 R CNN
-F 2 "" H 5650 4425 50  0001 C CNN
-F 3 "" H 5650 4425 50  0001 C CNN
-	1    5650 4225
+P 5650 4475
+F 0 "SW2" V 5696 4427 50  0000 R CNN
+F 1 "play" V 5605 4427 50  0000 R CNN
+F 2 "" H 5650 4675 50  0001 C CNN
+F 3 "" H 5650 4675 50  0001 C CNN
+	1    5650 4475
 	0    -1   -1   0
 $EndComp
-Wire Wire Line
-	5475 3525 5650 3525
-Wire Wire Line
-	5650 3525 5650 4025
 $Comp
 L power:GND #PWR02
 U 1 1 5BFF4A0B
-P 5650 4425
-F 0 "#PWR02" H 5650 4175 50  0001 C CNN
-F 1 "GND" H 5655 4252 50  0000 C CNN
-F 2 "" H 5650 4425 50  0001 C CNN
-F 3 "" H 5650 4425 50  0001 C CNN
-	1    5650 4425
-	1    0    0    -1
-$EndComp
-$Comp
-L power:GND #PWR05
+P 5650 4675
+F 0 "#PWR02" H 5650 4425 50  0001 C CNN
+F 1 "GND" H 5655 4502 50  0000 C CNN
+F 2 "" H 5650 4675 50  0001 C CNN
+F 3 "" H 5650 4675 50  0001 C CNN
+	1    5650 4675
+	1    0    0    -1
+$EndComp
+$Comp
+L power:GND #PWR06
 U 1 1 5BFF4A2E
-P 7350 3975
-F 0 "#PWR05" H 7350 3725 50  0001 C CNN
-F 1 "GND" H 7355 3802 50  0000 C CNN
-F 2 "" H 7350 3975 50  0001 C CNN
-F 3 "" H 7350 3975 50  0001 C CNN
-	1    7350 3975
-	1    0    0    -1
-$EndComp
-Wire Wire Line
-	7350 3750 7350 3975
+P 8375 4125
+F 0 "#PWR06" H 8375 3875 50  0001 C CNN
+F 1 "GND" H 8380 3952 50  0000 C CNN
+F 2 "" H 8375 4125 50  0001 C CNN
+F 3 "" H 8375 4125 50  0001 C CNN
+	1    8375 4125
+	1    0    0    -1
+$EndComp
+Wire Wire Line
+	8375 3900 8375 4125
 $Comp
 L device:CP C2
@@
 P 5950 3725
 F 0 "C2" H 6068 3771 50  0000 L CNN
-F 1 "22µF" H 6068 3680 50  0000 L CNN
+F 1 "33µF" H 6068 3680 50  0000 L CNN
 F 2 "" H 5988 3575 50  0001 C CNN
 F 3 "" H 5950 3725 50  0001 C CNN
@@
 	1    0    0    -1
 $EndComp
+$Comp
+L device:Speaker LS1
+U 1 1 5C003E50
+P 6950 3775
+F 0 "LS1" H 7120 3771 50  0000 L CNN
+F 1 "135R" H 7120 3680 50  0000 L CNN
+F 2 "" H 6950 3575 50  0001 C CNN
+F 3 "" H 6940 3725 50  0001 C CNN
+	1    6950 3775
+	1    0    0    -1
+$EndComp
+$Comp
+L power:GND #PWR04
+U 1 1 5C003EDE
+P 6750 4075
+F 0 "#PWR04" H 6750 3825 50  0001 C CNN
+F 1 "GND" H 6755 3902 50  0000 C CNN
+F 2 "" H 6750 4075 50  0001 C CNN
+F 3 "" H 6750 4075 50  0001 C CNN
+	1    6750 4075
+	1    0    0    -1
+$EndComp
+Wire Wire Line
+	6750 3625 6750 3775
+Wire Wire Line
+	6750 3875 6750 4075
+Wire Notes Line
+	7425 3250 7425 4675
+Text Notes 8050 4525 0    50   ~ 0
+option 2\n
+Text Label 7775 3775 0    50   ~ 0
+Eq1
+Text Label 6750 3650 0    50   ~ 0
+Eq1
+Text Notes 6050 4625 0    50   ~ 0
+durée de l'attaque 5*R1*C2\ndurée du déclin 5*(R2+GRe)*C2
+$Comp
+L device:LED D1
+U 1 1 5C0187FD
+P 5375 2850
+F 0 "D1" H 5367 2595 50  0000 C CNN
+F 1 "LED" H 5367 2686 50  0000 C CNN
+F 2 "" H 5375 2850 50  0001 C CNN
+F 3 "" H 5375 2850 50  0001 C CNN
+	1    5375 2850
+	-1   0    0    1
+$EndComp
+$Comp
+L device:R R1
+U 1 1 5C018B81
+P 4975 2850
+F 0 "R1" V 4768 2850 50  0000 C CNN
+F 1 "470R" V 4859 2850 50  0000 C CNN
+F 2 "" V 4905 2850 50  0001 C CNN
+F 3 "" H 4975 2850 50  0001 C CNN
+	1    4975 2850
+	0    1    1    0
+$EndComp
+Text Label 4825 2850 2    50   ~ 0
++Vdd
+Wire Wire Line
+	5125 2850 5225 2850
+Text Label 4175 3325 1    50   ~ 0
++Vdd
+Wire Wire Line
+	5475 3625 5650 3625
+$Comp
+L device:R R2
+U 1 1 5C019A4C
+P 5125 4200
+F 0 "R2" V 4918 4200 50  0000 C CNN
+F 1 "33k" V 5009 4200 50  0000 C CNN
+F 2 "" V 5055 4200 50  0001 C CNN
+F 3 "" H 5125 4200 50  0001 C CNN
+	1    5125 4200
+	0    1    1    0
+$EndComp
+Wire Wire Line
+	5475 3525 5525 3525
+Wire Wire Line
+	5525 3525 5525 2850
+Text Label 4975 4200 2    50   ~ 0
++Vdd
+Wire Wire Line
+	7775 3800 8375 3800
+Wire Wire Line
+	5650 3625 5650 4200
+Wire Wire Line
+	5275 4200 5650 4200
+Connection ~ 5650 4200
+Wire Wire Line
+	5650 4200 5650 4275
+Wire Notes Line
+	7425 3250 9050 3250
+Wire Notes Line
+	9050 3250 9050 4650
+Wire Notes Line
+	9050 4650 7450 4650
+Text Notes 5075 2475 0    79   ~ 0
+boite à musique
 $EndSCHEMATC
